File: Logic_Analyser_Breakout_40pin/Logic_Analyser_Breakout_40pin.kicad_pcb (KiCad board)
At the start: 2 copper layers, 32.4 x 52.1 mm, 4 parts, among them J1 40pin IC, J2 Analyser Left, J3 Analyser Right, J4 IC Socket

Commit message: Updated PCB artwork
Parts:
- moved J1 73.9 mm to (64.6, 39.6)
- moved J2 73.9 mm to (61.4, 39.6)
- moved J4 73.9 mm to (67.2, 39.6)
- moved J3 73.9 mm to (86.2, 39.6)
