File: Video_Buffer/RevB/Video_Buffer_RevB.kicad_pcb (KiCad board)
At the start: 2 copper layers, 21.5 x 11.7 mm, 13 parts, among them J1 +5V, J2 V_{IN}, J3 V_{OUT}, J4 GND, J5 GND, J6 GND Joint F, J7 GND Joint B, Q1 MMBT2222A

Commit message: Finalised for testing
Routing:
- net GND: track 29.1 -> 32.0 mm, vias 13 -> 10
- removed copper zone on B.Cu, net GND
Other:
- board text added: "100nF"
- board text added: "10µF"
- board text added: "222"
- board text added: "332"
- board text added: "751"
- board text added: "<--- Solder edge to inside of RF modulator can"
- board text added: "Brett Hallen, Oct 2026"
- board text added: "Clueless Video Buffer Oct 2026"
